File: myocell_s3/cpu_wroom_esp32.kicad_sch (KiCad schematic)
At the start: 16 parts, among them SW1 SW_Push, SW2 SW_Push, U4 ESP32-WROOM-E

Commit message: recovery commit
Parts:
- removed U4: ESP32-WROOM-E, RF_Module:ESP32-WROOM-32E, symbol espressif_github:ESP32-WROOM-E
- added U4: ESP32-S3-WROOM-2, RF_Module:ESP32-S3-WROOM-2, symbol myocell_s3:ESP32-S3-WROOM-2
- C24: value 0.1uF -> 1uF
- R16: value 10k -> 5.1k
Connections:
- net 3.3V: now also U4.2 (3v3)
- net EN: now also U4.3 (EN)
- net GND: now also U4. (GND41), U4.1 (GND1), U4.40 (GND40)
Other:
- moved on the sheet: C24, D8, R16, R32, SW1

Commit message: working on schematic
Connections:
- net IO0: now also U4.27 (IO0)
- net D-: now reaches U4.13 (IO19)
- net D+: now reaches U4.14 (IO20)
Other:
- title: ESP32 CPU -> ESP32-S3 CPU
- moved on the sheet: R17
Changed lines of the file:
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@@
 	(paper "A4")
 	(title_block
-		(title "ESP32 CPU")
-		(date "2024-10-17")
+		(title "ESP32-S3 CPU")
+		(date "2025-10-10")
 		(company "MIREA")
 	)
@@
 	(wire
 		(pts
-			(xy 134.62 77.47) (xy 149.86 77.47)
-		)
-		(stroke
-			(width 0)
-			(type default)
-		)
-	)
-	(wire
-		(pts
 			(xy 226.06 38.1) (xy 233.68 38.1)
 		)
@@
 	(wire
 		(pts
-			(xy 134.62 85.09) (xy 149.86 85.09)
-		)
-		(stroke
-			(width 0)
-			(type default)
-		)
-	)
-	(wire
-		(pts
-			(xy 134.62 69.85) (xy 149.86 69.85)
-		)
-		(stroke
-			(width 0)
-			(type default)
-		)
-	)
-	(wire
-		(pts
-			(xy 134.62 107.95) (xy 196.85 107.95)
+			(xy 152.4 85.09) (xy 167.64 85.09)
 		)
 		(stroke
@@
 	(wire
 		(pts
-			(xy 134.62 100.33) (xy 149.86 100.33)
+			(xy 152.4 100.33) (xy 167.64 100.33)
 		)
 		(stroke
@@
 	(wire
 		(pts
-			(xy 134.62 102.87) (xy 149.86 102.87)
+			(xy 152.4 102.87) (xy 167.64 102.87)
 		)
 		(stroke
@@
 	(wire
 		(pts
+			(xy 67.31 101.6) (xy 74.93 101.6)
+		)
+		(stroke
+			(width 0)
+			(type default)
+		)
+	)
+	(wire
+		(pts
 			(xy 38.1 77.47) (xy 44.45 77.47)
 		)
@@
 	(wire
 		(pts
-			(xy 134.62 87.63) (xy 139.7 87.63)
-		)
-		(stroke
-			(width 0)
-			(type default)
-		)
-	)
-	(wire
-		(pts
-			(xy 134.62 72.39) (xy 149.86 72.39)
+			(xy 120.65 101.6) (xy 125.73 101.6)
+		)
+		(stroke
+			(width 0)
+			(type default)
+		)
+	)
+	(wire
+		(pts
+			(xy 152.4 87.63) (xy 157.48 87.63)
 		)
 		(stroke
@@
 	(wire
 		(pts
+			(xy 67.31 99.06) (xy 74.93 99.06)
+		)
+		(stroke
+			(width 0)
+			(type default)
+		)
+	)
+	(wire
+		(pts
 			(xy 106.68 27.94) (xy 119.38 27.94)
 		)
@@
 	(wire
 		(pts
-			(xy 134.62 92.71) (xy 149.86 92.71)
+			(xy 152.4 92.71) (xy 167.64 92.71)
 		)
 		(stroke
@@
 	(wire
 		(pts
-			(xy 134.62 95.25) (xy 149.86 95.25)
-		)
-		(stroke
-			(width 0)
-			(type default)
-		)
-	)
-	(wire
-		(pts
-			(xy 134.62 97.79) (xy 149.86 97.79)
+			(xy 152.4 95.25) (xy 167.64 95.25)
+		)
+		(stroke
+			(width 0)
+			(type default)
+		)
+	)
+	(wire
+		(pts
+			(xy 152.4 97.79) (xy 167.64 97.79)
 		)
 		(stroke
@@
 	(wire
 		(pts
-			(xy 134.62 82.55) (xy 149.86 82.55)
+			(xy 152.4 82.55) (xy 167.64 82.55)
 		)
 		(stroke
@@
 	(wire
 		(pts
-			(xy 147.32 87.63) (xy 149.86 87.63)
+			(xy 165.1 87.63) (xy 167.64 87.63)
 		)
 		(stroke
@@
 	(wire
 		(pts
-			(xy 134.62 110.49) (xy 149.86 110.49)
+			(xy 152.4 110.49) (xy 167.64 110.49)
 		)
 		(stroke
@@
 			(width 0)
 			(type default)
+		)
+	)
+	(global_label "IO0"
+		(shape input)
+		(at 251.46 33.02 0)
+		(fields_autoplaced yes)
+		(effects
+			(font
+				(size 1.27 1.27)
+			)
+			(justify left)
+		)
+		(property "Intersheetrefs" "${INTERSHEET_REFS}"
+			(at 257.59 33.02 0)
+			(effects
+				(font
+					(size 1.27 1.27)
+				)
+				(justify left)
+				(hide yes)
+			)
 		)
 	)
@@
 		)
 	)
+	(global_label "IO0"
+		(shape input)
+		(at 125.73 101.6 0)
+		(fields_autoplaced yes)
+		(effects
+			(font
+				(size 1.27 1.27)
+			)
+			(justify left)
+		)
+		(property "Intersheetrefs" "${INTERSHEET_REFS}"
+			(at 131.86 101.6 0)
+			(effects
+				(font
+					(size 1.27 1.27)
+				)
+				(justify left)
+				(hide yes)
+			)
+		)
+	)
 	(global_label "EN"
 		(shape input)
@@
 		)
 	)
-	(hierarchical_label "TXD0"
-		(shape input)
-		(at 149.86 69.85 0)
-		(effects
-			(font
-				(size 1.27 1.27)
-			)
-			(justify left)
+	(hierarchical_label "D+"
+		(shape input)
+		(at 67.31 101.6 180)
+		(effects
+			(font
+				(size 1.27 1.27)
+			)
+			(justify right)
 		)
 	)
@@
 	(hierarchical_label "gpio22_pwdn"
 		(shape input)
-		(at 149.86 100.33 0)
+		(at 167.64 100.33 0)
 		(effects
 			(font
@@
 	(hierarchical_label "gpio4"
 		(shape input)
-		(at 149.86 82.55 0)
+		(at 167.64 82.55 0)
 		(effects
 			(font
@@
 	(hierarchical_label "gpio27"
 		(shape input)
-		(at 149.86 110.49 0)
+		(at 167.64 110.49 0)
 		(effects
 			(font
@@
 	(hierarchical_label "gpio19_vspi_miso"
 		(shape input)
-		(at 149.86 95.25 0)
+		(at 167.64 95.25 0)
 		(effects
 			(font
@@
 	(hierarchical_label "gpio21_start"
 		(shape input)
-		(at 149.86 97.79 0)
+		(at 167.64 97.79 0)
 		(effects
 			(font
@@
 		)
 	)
-	(hierarchical_label "RXD0"
-		(shape input)
-		(at 149.86 72.39 0)
-		(effects
-			(font
-				(size 1.27 1.27)
-			)
-			(justify left)
+	(hierarchical_label "D-"
+		(shape input)
+		(at 67.31 99.06 180)
+		(effects
+			(font
+				(size 1.27 1.27)
+			)
+			(justify right)
 		)
 	)
 	(hierarchical_label "3.3V"
 		(shape input)
-		(at 149.86 87.63 0)
+		(at 167.64 87.63 0)
 		(effects
 			(font
@@
 	(hierarchical_label "gpio5_vspi_ss"
 		(shape input)
-		(at 149.86 85.09 0)
+		(at 167.64 85.09 0)
 		(effects
 			(font
@@
 	(hierarchical_label "gpio18_vspi_sck"
 		(shape input)
-		(at 149.86 92.71 0)
+		(at 167.64 92.71 0)
 		(effects
 			(font
@@
 		)
 	)
-	(hierarchical_label "IO0"
-		(shape input)
-		(at 149.86 77.47 0)
-		(effects
-			(font
-				(size 1.27 1.27)
-			)
-			(justify left)
-		)
-	)
-	(hierarchical_label "IO0"
-		(shape input)
-		(at 251.46 33.02 0)
-		(effects
-			(font
-				(size 1.27 1.27)
-			)
-			(justify left)
-		)
-	)
 	(hierarchical_label "gpio23_vspi_mosi"
 		(shape input)
-		(at 149.86 102.87 0)
+		(at 167.64 102.87 0)
 		(effects
 			(font
@@
 	(symbol
 		(lib_id "Device:R_US")
-		(at 143.51 87.63 90)
+		(at 161.29 87.63 90)
 		(unit 1)
 		(exclude_from_sim no)
@@
 		(dnp no)
 		(property "Reference" "R17"
-			(at 145.288 86.614 90)
+			(at 163.068 86.614 90)
 			(effects
 				(font
@@
 		)
 		(property "Value" "10k"
-			(at 136.906 87.122 90)
+			(at 154.686 87.122 90)
 			(effects
 				(font
@@
 		)
 		(property "Footprint" "Resistor_SMD:R_0805_2012Metric_Pad1.20x1.40mm_HandSolder"
-			(at 143.764 86.614 90)
+			(at 161.544 86.614 90)
 			(effects
 				(font
@@
 		)
 		(property "Datasheet" "~"
-			(at 143.51 87.63 0)
+			(at 161.29 87.63 0)
 			(effects
 				(font
@@
 		)
 		(property "Description" ""
-			(at 143.51 87.63 0)
-			(effects
-				(font
+			(at 161.29 87.63 0)
+			(effects
+				(font

Commit message: working on schematic
Parts:
- added C57: 10pF, Capacitor_SMD:C_0805_2012Metric_Pad1.18x1.45mm_HandSolder, symbol Device:C
- added R51, R52, R53, R54: 20, Resistor_SMD:R_0805_2012Metric_Pad1.20x1.40mm_HandSolder, symbol Device:R_US
Connections:
- net GND: now also C57.1
- net gpio4: now also U4.4 (IO4)
- net at U4.18 (IO10): now also R51.2
- net at U4.19 (IO11): now also R52.2
- net at U4.20 (IO12): now also R53.2
- net at U4.21 (IO13): now also R54.2
- net start: now reaches U4.22 (IO14)
- net clk: now reaches U4.23 (IO21)
- net reset: now reaches U4.24 (IO47)
- net pwdn: now reaches U4.25 (IO48)
- new net fspi_clk: C57.2, R53.1
- new net fspi_cs0: R51.1
- new net fspi_miso: R54.1
- new net fspi_mosi: R52.1
Other:
- note added: "Interface 4c (see Table 2-4) is multiplexed with GPIO9 ~ GPIO14, RTC_GPIO9 ~ RTC_GPIO14, Touch Sensor interface, SAR ADC interface, and SPI interfaces 4d and 4g via IO MUX. It is the SPI2 main interface for fast SPI connection (ESP32-S3 Series Datasheet)"
- note added: "Technical Reference Chapter 30 SPI Controller"

Commit message: working on schematic transfer
Parts:
- removed C28, C30: 0.1uF, Capacitor_SMD:C_0805_2012Metric_Pad1.18x1.45mm_HandSolder, symbol Device:C
- removed D1, D2: WS2812B, LED_SMD:LED_WS2812B_PLCC4_5.0x5.0mm_P3.2mm, symbol LED:WS2812B
- removed R17, R18: 10k, Resistor_SMD:R_0805_2012Metric_Pad1.20x1.40mm_HandSolder, symbol Device:R_US
- added R55, R56: 10k, Resistor_SMD:R_0805_2012Metric_Pad1.20x1.40mm_HandSolder, symbol Device:R_US
Connections:
- net GND: now also R55.1, R56.2
- net clk: now also U4.24 (IO47); no longer U4.23 (IO21)
- net pwdn: now also U4.12 (IO8); no longer U4.25 (IO48)
- net reset: now also U4.25 (IO48); no longer U4.24 (IO47)
- net start: now also U4.23 (IO21); no longer U4.22 (IO14)
- net IO5: now reaches R32.2
- net IO5: now also U4.5 (IO5)
- net at U4.15 (IO3): now also R56.1
- net at U4.16 (IO46): now also R55.2
- net bat_mon: now reaches U4.7 (IO7)
- net gpio4: no longer names the net of U4.4 (IO4)
Other:
- note added: "IO46 should be 0 @RESET to enable joint download boot default: weak pull-down https://documentation.espressif.com/esp32-s3-wroom-2_datasheet_en.pdf https://.../en/latest/esp32s3/schematic-checklist.html"
- note removed: "RGB Led"
- moved on the sheet: C24, C29, C57, D8, R16, R32, R51, R52, R53, R54, SW1, SW2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

Commit message: RLDINV still unconnected
Parts:
- SW1, SW2: footprint Button_Switch_SMD:SW_SPST_PTS645 -> Button_Switch_SMD:SW_SPST_PTS645Sx43SMTR92
Connections:
- net GND: now also U4.41 (GND41); no longer U4. (GND41)
Changed lines of the file:
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@@
 			)
 		)
-		(property "Description" ""
+		(property "Description" "Unpolarized capacitor"
 			(at 46.99 44.45 0)
 			(effects
@@
 			)
 		)
-		(property "Description" ""
+		(property "Description" "Power symbol creates a global label with name \"GND\" , ground"
 			(at 22.86 46.99 0)
 			(effects
@@
 			)
 		)
-		(property "Description" ""
+		(property "Description" "Resistor, US symbol"
 			(at 85.09 111.76 0)
 			(effects
@@
 			)
 		)
-		(property "Description" ""
+		(property "Description" "Light emitting diode"
+			(at 31.75 97.79 0)
+			(effects
+				(font
+					(size 1.27 1.27)
+				)
+				(hide yes)
+			)
+		)
+		(property "Sim.Pins" "1=K 2=A"
 			(at 31.75 97.79 0)
 			(effects
@@
 			)
 		)
-		(property "Description" ""
+		(property "Description" "Resistor, US symbol"
 			(at 110.49 116.84 0)
 			(effects
@@
 			)
 		)
-		(property "Footprint" "Button_Switch_SMD:SW_SPST_PTS645"
+		(property "Footprint" "Button_Switch_SMD:SW_SPST_PTS645Sx43SMTR92"
 			(at 31.75 34.29 0)
 			(effects
@@
 			)
 		)
-		(property "Description" ""
+		(property "Description" "Power symbol creates a global label with name \"GND\" , ground"
 			(at 82.55 63.5 0)
 			(effects
@@
 			)
 		)
-		(property "Description" ""
+		(property "Description" "Unpolarized capacitor"
 			(at 116.84 139.7 0)
 			(effects
@@
 			)
 		)
-		(property "Description" ""
+		(property "Description" "Power symbol creates a global label with name \"GND\" , ground"
 			(at 120.65 139.7 0)
 			(effects
@@
 			)
 		)
-		(property "Description" ""
+		(property "Description" "Resistor, US symbol"
 			(at 102.87 116.84 0)
 			(effects
@@
 			)
 		)
-		(property "Description" ""
+		(property "Description" "Resistor, US symbol"
 			(at 105.41 116.84 0)
 			(effects
@@
 			)
 		)
-		(property "Description" ""
+		(property "Description" "Unpolarized capacitor"
 			(at 39.37 73.66 0)
 			(effects
@@
 			)
 		)
-		(property "Description" ""
+		(property "Description" "Resistor, US symbol"
 			(at 38.1 90.17 0)
 			(effects
@@
 			)
 		)
-		(property "Description" ""
+		(property "Description" "Unpolarized capacitor"
 			(at 106.68 31.75 0)
 			(effects
@@
 			)
 		)
-		(property "Description" ""
+		(property "Description" "Resistor, US symbol"
 			(at 46.99 33.02 0)
 			(effects
@@
 			)
 		)
-		(property "Footprint" "Button_Switch_SMD:SW_SPST_PTS645"
+		(property "Footprint" "Button_Switch_SMD:SW_SPST_PTS645Sx43SMTR92"
 			(at 39.37 63.5 0)
 			(effects
@@
 			)
 		)
-		(property "Description" ""
+		(property "Description" "Power symbol creates a global label with name \"GND\" , ground"
 			(at 137.16 63.5 0)
 			(effects
@@
 			)
 		)
-		(property "Description" ""
+		(property "Description" "Power symbol creates a global label with name \"GND\" , ground"
 			(at 31.75 104.14 0)
 			(effects
@@
 			)
 		)
-		(property "Description" ""
+		(property "Description" "Power symbol creates a global label with name \"GND\" , ground"
 			(at 110.49 55.88 0)
 			(effects
@@
 			)
 		)
-		(property "Description" ""
+		(property "Description" "Unpolarized capacitor"
 			(at 119.38 31.75 0)
 			(effects
@@
 		(pin "20"
 		)
-		(pin ""
+		(pin "41"
 		)
 		(pin "22"
@@
 			)
 		)
-		(property "Description" ""
+		(property "Description" "Power symbol creates a global label with name \"GND\" , ground"
 			(at 97.79 120.65 0)
 			(effects
@@
 			)
 		)
-		(property "Description" ""
+		(property "Description" "Resistor, US symbol"
 			(at 97.79 116.84 0)
 			(effects
@@
 			)
 		)
-		(property "Description" ""
+		(property "Description" "Resistor, US symbol"
 			(at 107.95 116.84 0)
 			(effects
@@
 			)
 		)
-		(property "Description" ""
+		(property "Description" "Power symbol creates a global label with name \"GND\" , ground"
 			(at 46.99 49.53 0)
 			(effects
@@
 			)
 		)
-		(property "Description" ""
+		(property "Description" "Power symbol creates a global label with name \"GND\" , ground"
 			(at 106.68 38.1 0)
 			(effects
@@
 			)
 		)
-		(property "Description" ""
+		(property "Description" "Power symbol creates a global label with name \"GND\" , ground"
 			(at 27.94 77.47 0)
 			(effects
@@
 			)
 		)
-		(property "Description" ""
+		(property "Description" "Power symbol creates a global label with name \"GND\" , ground"
 			(at 81.28 111.76 0)
 			(effects

Commit message: drdy fixed
Parts:
- removed C57: 10pF, Capacitor_SMD:C_0805_2012Metric_Pad1.18x1.45mm_HandSolder, symbol Device:C
Connections:
- net drdy: now reaches U4.22 (IO14)
Changed lines of the file:
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@@
-	)
-	(junction
-		(at 107.95 139.7)
-		(diameter 0)
-		(color 0 0 0 0)
 	)
 	(junction
@@
 	(wire
 		(pts
+			(xy 113.03 109.22) (xy 113.03 114.3)
+		)
+		(stroke
+			(width 0)
+			(type default)
+		)
+	)
+	(wire
+		(pts
 			(xy 95.25 109.22) (xy 95.25 111.76)
 		)
@@
 	(wire
 		(pts
-			(xy 107.95 120.65) (xy 107.95 139.7)
+			(xy 107.95 120.65) (xy 107.95 143.51)
 		)
 		(stroke
@@
 	(wire
 		(pts
-			(xy 107.95 139.7) (xy 107.95 143.51)
-		)
-		(stroke
-			(width 0)
-			(type default)
-		)
-	)
-	(wire
-		(pts
 			(xy 46.99 49.53) (xy 46.99 48.26)
 		)
@@
 		(pts
 			(xy 120.65 109.22) (xy 120.65 114.3)
-		)
-		(stroke
-			(width 0)
-			(type default)
-		)
-	)
-	(wire
-		(pts
-			(xy 107.95 139.7) (xy 113.03 139.7)
 		)
 		(stroke
@@
 		(shape input)
 		(at 120.65 114.3 270)
+		(effects
+			(font
+				(size 1.27 1.27)
+			)
+			(justify right)
+		)
+	)
+	(hierarchical_label "drdy"
+		(shape input)
+		(at 113.03 114.3 270)
 		(effects
 			(font
@@
 					(unit 1)
 				)
-			)
-		)
-	)
-	(symbol
-		(lib_id "Device:C")
-		(at 116.84 139.7 270)
-		(unit 1)
-		(exclude_from_sim no)
-		(in_bom yes)
-		(on_board yes)
-		(dnp no)
-		(property "Reference" "C57"
-			(at 117.094 132.588 0)
-			(effects
-				(font
-					(size 1.27 1.27)
-				)
-				(justify left)
-			)
-		)
-		(property "Value" "10pF"
-			(at 115.062 131.572 0)
-			(effects
-				(font
-					(size 1.27 1.27)
-				)
-				(justify left)
-			)
-		)
-		(property "Footprint" "Capacitor_SMD:C_0805_2012Metric_Pad1.18x1.45mm_HandSolder"
-			(at 113.03 140.6652 0)
-			(effects
-				(font
-					(size 1.27 1.27)
-				)
-				(hide yes)
-			)
-		)
-		(property "Datasheet" "~"
-			(at 116.84 139.7 0)
-			(effects
-				(font
-					(size 1.27 1.27)
-				)
-				(hide yes)
-			)
-		)
-		(property "Description" "Unpolarized capacitor"
-			(at 116.84 139.7 0)
-			(effects
-				(font
-					(size 1.27 1.27)
-				)
-				(hide yes)
-			)
-		)
-		(pin "1"
-		)
-		(pin "2"
-		)
-		(instances
-			(project "myocell_s3"
-				(path "/871ff10b-bde5-471c-b91a-de58aa271388/1fb257a1-4b3b-418e-bb46-683d94c5ed44"
-					(reference "C57")
-					(unit 1)
-				)
-			)
-		)
-	)
-	(symbol
-		(lib_id "power:GND")
-		(at 120.65 139.7 90)
-		(unit 1)
-		(exclude_from_sim no)
-		(in_bom yes)
-		(on_board yes)
-		(dnp no)
-		(fields_autoplaced yes)
-		(property "Reference" "#PWR044"
-			(at 127 139.7 0)
-			(effects
-				(font
-					(size 1.27 1.27)
-				)
-				(hide yes)
-			)
-		)
-		(property "Value" "GND"
-			(at 124.46 139.6999 90)
-			(effects
-				(font
-					(size 1.27 1.27)
-				)
-				(justify right)
-			)
-		)
-		(property "Footprint" ""
-			(at 120.65 139.7 0)
-			(effects
-				(font
-					(size 1.27 1.27)
-				)
-				(hide yes)
-			)
-		)
-		(property "Datasheet" ""
-			(at 120.65 139.7 0)
-			(effects
-				(font
-					(size 1.27 1.27)
-				)
-				(hide yes)
-			)
-		)
-		(property "Description" "Power symbol creates a global label with name \"GND\" , ground"
-			(at 120.65 139.7 0)
-			(effects
-				(font
-					(size 1.27 1.27)
-				)
-				(hide yes)
-			)
-		)
-		(pin "1"
-		)
-		(instances
-			(project "myocell_s3"
-				(path "/871ff10b-bde5-471c-b91a-de58aa271388/1fb257a1-4b3b-418e-bb46-683d94c5ed44"
-					(reference "#PWR044")
-					(unit 1)
-				)

Commit message: routing
Connections:
- net IO1: now reaches U4.39 (IO1)
- net IO1: now also R32.2
- net IO5: no longer names the net of U4.5 (IO5)
- net IO5: no longer R32.2
Changed lines of the file:
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@@
+	(wire
+		(pts
+			(xy 133.35 66.04) (xy 138.43 66.04)
+		)
+		(stroke
+			(width 0)
+			(type default)
+		)
+	)
 	(wire
 		(pts
@@
 	(wire
 		(pts
-			(xy 82.55 73.66) (xy 87.63 73.66)
-		)
-		(stroke
-			(width 0)
-			(type default)
-		)
-	)
-	(wire
-		(pts
 			(xy 120.65 109.22) (xy 120.65 114.3)
 		)
@@
 			(width 0)
 			(type default)
-		)
-	)
-	(global_label "IO5"
-		(shape input)
-		(at 82.55 73.66 180)
-		(fields_autoplaced yes)
-		(effects
-			(font
-				(size 1.27 1.27)
-			)
-			(justify right)
-		)
-		(property "Intersheetrefs" "${INTERSHEET_REFS}"
-			(at 76.42 73.66 0)
-			(effects
-				(font
-					(size 1.27 1.27)
-				)
-				(justify right)
-				(hide yes)
-			)
 		)
 	)
@@
 		)
 	)
+	(global_label "IO1"
+		(shape input)
+		(at 138.43 66.04 0)
+		(fields_autoplaced yes)
+		(effects
+			(font
+				(size 1.27 1.27)
+			)
+			(justify left)
+		)
+		(property "Intersheetrefs" "${INTERSHEET_REFS}"
+			(at 144.56 66.04 0)
+			(effects
+				(font
+					(size 1.27 1.27)
+				)
+				(justify left)
+				(hide yes)
+			)
+		)
+	)
 	(global_label "EN"
 		(shape input)
@@
 		)
 	)
-	(global_label "IO5"
+	(global_label "IO1"
 		(shape input)
 		(at 50.8 90.17 0)
