File: emg_filter/emg-lab-passive-filter-dif-1.kicad_sch (KiCad schematic)
At the start: 20 parts, among them U1 INA331

Commit message: add transient settings
Parts:
- V3: value 1.6 -> 3.2
Other:
- note added: "Load"
Changed lines of the file:
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@@
+		)
+	)
+	(text "Load"
+		(exclude_from_sim no)
+		(at 200.914 61.976 0)
+		(effects
+			(font
+				(size 1.27 1.27)
+			)
 		)
 	)
@@
 			)
 		)
-		(property "Sim.Params" "dc=0 ampl=1 f=1k ac=1"
+		(property "Sim.Params" "dc=0 ampl=0.1 f=100 ac=1"
 			(at 24.384 53.086 0)
 			(effects
@@
 			)
 		)
-		(property "Value" "1.6"
+		(property "Value" "3.2"
 			(at 146.05 84.9601 0)
 			(effects
